File: brain_PCB/brain_PCB.kicad_sch (KiCad schematic)
At the start: 0 parts

Commit message: brain PCB schematic in progress: power pins, decoupling caps, VCAP, crystals, reset, boot, SWD, UART, analog sensors, temp probes
Parts:
- added C1, C2, C3: 100nF, symbol Device:C
- added C4, C5: 20pF, symbol Device:C
- added C6, decoupl_C1, decoupl_C10, decoupl_C11, decoupl_C12, decoupl_C13, decoupl_C2, decoupl_C3, decoupl_C4, decoupl_C5, decoupl_C6, decoupl_C7, decoupl_C8, decoupl_C9: 100nf, symbol Device:C
- added C7, VCAP_C1: 2.2µF, symbol Device:C
- added C8, C9: 10pF, symbol Device:C
- added J1, J2, J3: Conn_01x02, symbol Connector_Generic:Conn_01x02
- added J4, J5, UARTdebugHeader1: Conn_01x03, symbol Connector_Generic:Conn_01x03
- added R1, R2, R3: 1k, symbol Device:R
- added R4: 10k, symbol Device:R
- added R5, R6: 4.7k, symbol Device:R
- added SW1: SW_Push, symbol Switch:SW_Push
- added SWDdebugHeader1: Conn_01x04, symbol Connector_Generic:Conn_01x04
- added U1: STM32H753ZITx, Package_QFP:LQFP-144_20x20mm_P0.5mm, symbol MCU_ST_STM32H7:STM32H753ZITx
- added Y1, Y2: Crystal, symbol Device:Crystal
- added rescaps_C1, rescaps_C2: 10µF, symbol Device:C
Connections:
- new net: C4.2, U1.23 (PH0), Y1.1
- new net: C5.1, U1.24 (PH1), Y1.2
- new net: U1.106 (VCAP), VCAP_C1.2
- new net: R4.2, U1.138 (BOOT0)
- new net: C6.2, SW1.2, U1.25 (NRST)
- new net: C7.2, U1.71 (VCAP)
- new net: C8.2, U1.8 (PC14), Y2.2
- new net: C9.1, U1.9 (PC15), Y2.1
- new net +3V3: J4.3 (Pin_3), J5.3 (Pin_3), R5.2, R6.2, SWDdebugHeader1.1 (Pin_1), U1.108 (VDD), U1.121 (VDD), U1.131 (VDD), U1.143 (PDR_ON), U1.144 (VDD), U1.17 (VDD), U1.30 (VDD), U1.39 (VDD), U1.52 (VDD), U1.6 (VBAT), U1.62 (VDD), U1.72 (VDD), U1.84 (VDD), decoupl_C1.2, decoupl_C10.2, decoupl_C11.2, decoupl_C12.2, decoupl_C13.2, decoupl_C2.2, decoupl_C3.2, decoupl_C4.2, decoupl_C5.2, decoupl_C6.2, decoupl_C7.2, decoupl_C8.2, decoupl_C9.2, rescaps_C1.2, rescaps_C2.2
- new net GND: C1.2, C2.2, C3.2, C4.1, C5.2, C6.1, C7.1, C8.1, C9.2, J1.2 (Pin_2), J2.2 (Pin_2), J3.2 (Pin_2), J4.1 (Pin_1), J5.1 (Pin_1), R4.1, SW1.1, SWDdebugHeader1.4 (Pin_4), U1.107 (VSS), U1.120 (VSS), U1.130 (VSS), U1.16 (VSS), U1.31 (VSSA), U1.38 (VSS), U1.51 (VSS), U1.61 (VSS), U1.83 (VSS), U1.94 (VSS), UARTdebugHeader1.1 (Pin_1), VCAP_C1.1, decoupl_C1.1, decoupl_C10.1, decoupl_C11.1, decoupl_C12.1, decoupl_C13.1, decoupl_C2.1, decoupl_C3.1, decoupl_C4.1, decoupl_C5.1, decoupl_C6.1, decoupl_C7.1, decoupl_C8.1, decoupl_C9.1, rescaps_C1.1, rescaps_C2.1
- new net LEVEL_IN: J3.1 (Pin_1), R3.2
- new net LEVEL_PWR: U1.87 (PG2)
- new net PA6: C1.1, R1.1, U1.42 (PA6)
- new net PC0: C2.1, R2.1, U1.26 (PC0)
- new net PC3_C: C3.1, R3.1, U1.29 (PC3_C)
- new net PF1: J4.2 (Pin_2), R5.1, U1.11 (PF1)
- new net PF2: J5.2 (Pin_2), R6.1, U1.12 (PF2)
- new net PH_IN: J2.1 (Pin_1), R2.2
- new net SWCLK: SWDdebugHeader1.3 (Pin_3), U1.109 (PA14)
- new net SWDIO: SWDdebugHeader1.2 (Pin_2), U1.105 (PA13)
- new net TDS_IN: J1.1 (Pin_1), R1.2
- new net UART_RX: U1.78 (PD9), UARTdebugHeader1.3 (Pin_3)
- new net UART_TX: U1.77 (PD8), UARTdebugHeader1.2 (Pin_2)

Commit message: full schematic complete; minor warnings regarding labels
Parts:
- added C10: 1µF, symbol Device:C
- added C11: 100nF, symbol Device:C
- added FB1: FerriteBead, symbol Device:FerriteBead
- added J6: Conn_01x04, symbol Connector_Generic:Conn_01x04
- added J7: Conn_01x14, symbol Connector_Generic:Conn_01x14
- added J8: Conn_01x06, symbol Connector_Generic:Conn_01x06
- added J9: Conn_01x08, symbol Connector_Generic:Conn_01x08
- added R10, R11, R12, R13, R14, R15, R16: 10k, symbol Device:R
- added R7, R8: 1.9k, symbol Device:R
- added R9: 47, symbol Device:R
Connections:
- net +3V3: now also FB1.1, J6.1 (Pin_1), J7.1 (Pin_1), R14.1, R15.1, R16.1, R7.2, R8.2
- net GND: now also C10.2, C11.2, J6.4 (Pin_4), J7.2 (Pin_2), J8.1 (Pin_1), J9.1 (Pin_1), R10.1, R11.1, R12.1, R13.1
- net LCD_D0: now reaches U1.114 (PD0)
- net LCD_D0: now also J7.7 (Pin_7)
- net LCD_D1: now reaches U1.115 (PD1)
- net LCD_D1: now also J7.8 (Pin_8)
- net LCD_D2: now reaches U1.116 (PD2)
- net LCD_D2: now also J7.9 (Pin_9)
- net LCD_D3: now reaches U1.117 (PD3)
- net LCD_D3: now also J7.10 (Pin_10)
- net LCD_D4: now reaches U1.118 (PD4)
- net LCD_D4: now also J7.11 (Pin_11)
- net LCD_D5: now reaches U1.119 (PD5)
- net LCD_D5: now also J7.12 (Pin_12)
- net LCD_D6: now reaches U1.122 (PD6)
- net LCD_D6: now also J7.13 (Pin_13)
- net LCD_D7: now reaches U1.123 (PD7)
- net LCD_D7: now also J7.14 (Pin_14)
- net SCL: now reaches U1.139 (PB8)
- net SCL: now also J6.2 (Pin_2), R7.1
- net SDA: now reaches U1.140 (PB9)
- net SDA: now also J6.3 (Pin_3), R8.1
- net VDDA: now reaches U1.32 (VREF+)
- net VDDA: now also U1.33 (VDDA), U1.95 (VDD33_USB), C10.1, C11.1, FB1.2
- net BLUE_PWM: now reaches U1.47 (PB1)
- net BLUE_PWM: now also J8.2 (Pin_2)
- net HEATER: now reaches U1.58 (PE7)
- net HEATER: now also J9.2 (Pin_2), R10.2
- net COOLER: now reaches U1.59 (PE8)
- net COOLER: now also J9.3 (Pin_3), R11.2
- net PH_DOWN: now reaches U1.63 (PE10)
- net PH_DOWN: now also J9.5 (Pin_5), R13.2
- net RED_PWM: now reaches U1.64 (PE11)
- net RED_PWM: now also J8.3 (Pin_3)
- net PH_UP: now reaches U1.65 (PE12)
- net PH_UP: now also J9.4 (Pin_4), R12.2
- net NIR_PWM: now reaches U1.66 (PE13)
- net NIR_PWM: now also J8.4 (Pin_4)
- net FAN_PWM: now reaches U1.67 (PE14)
- net FAN_PWM: now also J8.6 (Pin_6)
- net FLORA_MICRO: now reaches U1.68 (PE15)
- net FLORA_MICRO: now also J9.6 (Pin_6), R14.2
- net FLORA_BLOOM: now reaches U1.69 (PB10)
- net FLORA_BLOOM: now also J9.8 (Pin_8), R16.2
- net FLORA_GROW: now reaches U1.70 (PB11)
- net FLORA_GROW: now also J9.7 (Pin_7), R15.2
- net WHITE_PWM: now reaches U1.81 (PD12)
- net WHITE_PWM: now also J8.5 (Pin_5)
- net LCD_RST: now reaches U1.96 (PC6)
- net LCD_RST: now also J7.3 (Pin_3)
- net LCD_CD: now reaches U1.97 (PC7)
- net LCD_CD: now also J7.4 (Pin_4)
- net LCD_CS: now reaches U1.98 (PC8)
- net LCD_CS: now also J7.5 (Pin_5)
- net LCD_WR: now reaches U1.99 (PC9)
- net LCD_WR: now also R9.2
- new net: J7.6 (Pin_6), R9.1
Other:
- moved on the sheet: C1, C2, C3, C4, C5, C6, C7, C8, C9, J1, J2, J3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

Commit message: brain PCB schematic: footprints assigned, ready for PCB layout
Parts:
- added J10: Conn_01x02, Connector_PinHeader_2.54mm:PinHeader_1x02_P2.54mm_Vertical, symbol Connector_Generic:Conn_01x02
- C1, C10, C11, C2, C3, C4, C5, C6, C7, C8, C9, VCAP_C1, decoupl_C1, decoupl_C10, decoupl_C11, decoupl_C12, decoupl_C13, decoupl_C2, decoupl_C3, decoupl_C4, decoupl_C5, decoupl_C6, decoupl_C7, decoupl_C8, decoupl_C9, rescaps_C1, rescaps_C2: footprint (none) -> Capacitor_SMD:C_0402_1005Metric
- FB1: footprint (none) -> Inductor_SMD:L_0402_1005Metric
- J1, J2: footprint (none) -> Connector_PinHeader_2.54mm:PinHeader_1x02_P2.54mm_Vertical
- J3: footprint (none) -> Connector_PinHeader_2.54mm:PinHeader_1x01_P2.54mm_Vertical
- J4, J5, UARTdebugHeader1: footprint (none) -> Connector_PinHeader_2.54mm:PinHeader_1x03_P2.54mm_Vertical
- J6, SWDdebugHeader1: footprint (none) -> Connector_PinHeader_2.54mm:PinHeader_1x04_P2.54mm_Vertical
- J7: footprint (none) -> Connector_PinHeader_2.54mm:PinHeader_1x14_P2.54mm_Vertical
- J8: footprint (none) -> Connector_PinHeader_2.54mm:PinHeader_1x06_P2.54mm_Vertical
- J9: footprint (none) -> Connector_PinHeader_2.54mm:PinHeader_1x08_P2.54mm_Vertical
- R1, R10, R11, R12, R13, R14, R15, R16, R2, R3, R4, R5, R6, R7, R8, R9: footprint (none) -> Resistor_SMD:R_0402_1005Metric
- SW1: footprint (none) -> Button_Switch_SMD:SW_SPST_PTS645Sx43SMTR92
- Y1: value Crystal -> 8 MHz; footprint (none) -> Crystal:Crystal_SMD_3225-4Pin_3.2x2.5mm
- Y2: value Crystal -> 32.768 kHz; footprint (none) -> Crystal:Crystal_SMD_3215-2Pin_3.2x1.5mm
Connections:
- net +3V3: now also J10.1 (Pin_1)
- net GND: now also J10.2 (Pin_2)

Commit message: initial PCB placementt
Parts:
- J3: footprint Connector_PinHeader_2.54mm:PinHeader_1x01_P2.54mm_Vertical -> Connector_PinHeader_2.54mm:PinHeader_1x02_P2.54mm_Vertical
Changed lines of the file:
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@@
 			)
 		)
-		(property "Footprint" "Connector_PinHeader_2.54mm:PinHeader_1x01_P2.54mm_Vertical"
+		(property "Footprint" "Connector_PinHeader_2.54mm:PinHeader_1x02_P2.54mm_Vertical"
 			(at 25.4 125.73 0)
 			(hide yes)
