File: brain_PCB/brain_PCB.kicad_sch (KiCad schematic)
At the start: 60 parts, among them J1 Conn_01x02, J10 Conn_01x02, J2 Conn_01x02, J3 Conn_01x02, J4 Conn_01x03, J5 Conn_01x03, J6 Conn_01x04, J7 Conn_01x14, J8 Conn_01x06, J9 Conn_01x08, SW1 SW_Push, U1 STM32H753ZITx, Y1 8 MHz, Y2 32.768 kHz

Commit message: brain PCB routing complete: GND pours on outer layers, stitching vias, SI fixes; electrical DRC clean
Parts:
- Y1: symbol Device:Crystal -> Device:Crystal_GND24
Connections:
- net GND: now also Y1.2 (G), Y1.4 (G)
- net LCD_CD: now also U1.125 (PG10); no longer U1.97 (PC7)
- net LCD_CS: now also U1.126 (PG11); no longer U1.98 (PC8)
- net LCD_RST: now also U1.124 (PG9); no longer U1.96 (PC6)
- net LCD_WR: now also U1.127 (PG12); no longer U1.99 (PC9)
- net at C5.1, U1.24 (PH1): now also Y1.3; no longer Y1.2
- no-connect marks 0 -> 4
Changed lines of the file:
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@@
 		)
 	)
-	(label "LCD_CS"
-		(at 237.49 142.24 0)
-		(effects
-			(font
-				(size 1.27 1.27)
-			)
-			(justify left bottom)
-		)
-	)
 	(label "FLORA_MICRO"
 		(at 149.86 187.96 180)
@@
 		)
 	)
-	(label "LCD_WR"
-		(at 237.49 144.78 0)
-		(effects
-			(font
-				(size 1.27 1.27)
-			)
-			(justify left bottom)
-		)
-	)
 	(label "LCD_D4"
 		(at 38.1 240.03 0)
@@
 		)
 	)
-	(label "LCD_CD"
-		(at 237.49 139.7 0)
-		(effects
-			(font
-				(size 1.27 1.27)
-			)
-			(justify left bottom)
-		)
-	)
 	(label "powerIn"
 		(at 71.12 29.21 180)
@@
 		)
 	)
-	(label "LCD_RST"
-		(at 237.49 137.16 0)
-		(effects
-			(font
-				(size 1.27 1.27)
-			)
-			(justify left bottom)
-		)
-	)
 	(label "FLORA_MICRO"
 		(at 139.7 251.46 180)
@@
 	)
 	(symbol
-		(lib_id "Device:Crystal")
+		(lib_id "Device:Crystal_GND24")
 		(at 156.21 57.15 270)
 		(unit 1)
@@
 		(pin "2"
 		)
+		(pin "3"
+		)
+		(pin "4"
+		)
 		(instances
 			(project "brain_PCB"
@@
 		)
 	)
+	(symbol
+		(lib_id "power:GND")
+		(at 151.13 57.15 0)
+		(unit 1)
+		(body_style 1)
+		(exclude_from_sim no)
+		(in_bom yes)
+		(on_board yes)
+		(in_pos_files yes)
+		(dnp no)
+		(fields_autoplaced yes)
+		(property "Reference" "#PWR089"
+			(at 151.13 63.5 0)
+			(hide yes)
+			(show_name no)
+			(do_not_autoplace no)
+			(effects
+				(font
+					(size 1.27 1.27)
+				)
+			)
+		)
+		(property "Value" "GND"
+			(at 151.13 61.595 0)
+			(show_name no)
+			(do_not_autoplace no)
+			(effects
+				(font
+					(size 1.27 1.27)
+				)
+			)
+		)
+		(property "Footprint" ""
+			(at 151.13 57.15 0)
+			(hide yes)
+			(show_name no)
+			(do_not_autoplace no)
+			(effects
+				(font
+					(size 1.27 1.27)
+				)
+			)
+		)
+		(property "Datasheet" ""
+			(at 151.13 57.15 0)
+			(hide yes)
+			(show_name no)
+			(do_not_autoplace no)
+			(effects
+				(font
+					(size 1.27 1.27)
+				)
+			)
+		)
+		(property "Description" "Power symbol creates a global label with name \"GND\" , ground"
+			(at 151.13 57.15 0)
+			(hide yes)
+			(show_name no)
+			(do_not_autoplace no)
+			(effects
+				(font
+					(size 1.27 1.27)
+				)
+			)
+		)
+		(pin "1"
+		)
+		(instances
+			(project "brain_PCB"
+				(path "/4bb3d8ed-a62e-4677-afe9-da4a1eb55537"
+					(reference "#PWR089")
+					(unit 1)
+				)
+			)
+		)
+	)
+	(label "LCD_RST"
+		(at 161.29 86.36 180)
+		(effects
+			(font
+				(size 1.27 1.27)
+			)
+			(justify right bottom)
+		)
+	)
+	(label "LCD_CD"
+		(at 161.29 88.9 180)
+		(effects
+			(font
+				(size 1.27 1.27)
+			)
+			(justify right bottom)
+		)
+	)
+	(label "LCD_CS"
+		(at 161.29 91.44 180)
+		(effects
+			(font
+				(size 1.27 1.27)
+			)
+			(justify right bottom)
+		)
+	)
+	(label "LCD_WR"
+		(at 161.29 93.98 180)
+		(effects
+			(font
+				(size 1.27 1.27)
+			)
+			(justify right bottom)
+		)
+	)
+	(no_connect
+		(at 237.49 137.16)
+	)
+	(no_connect
+		(at 237.49 139.7)
+	)
+	(no_connect
+		(at 237.49 142.24)
+	)
+	(no_connect
+		(at 237.49 144.78)
+	)
 	(sheet_instances

Commit message: all boards routed: light rev B (SOT-23 switches, protected input), pump rev B (CSD18540 MOSFETs), power rev A1 (parts selected), brain Micro-Fit connectors + display on edge; whitelist gitignore
Light, power and pump pass DRC and ERC clean. Brain routed with 0 unconnected; remaining warnings are dangling vias, thin silk text and missing no-connect flags. All cable connectors standardized to Molex Micro-Fit 3.0. Repo now tracks only the KiCad project files, design rules, local libraries and brain 3D models.
Parts:
- added C12: 100nF, Capacitor_SMD:C_0402_1005Metric, symbol Device:C
- added C13: 1uF, Capacitor_SMD:C_0402_1005Metric, symbol Device:C
- added J11: USB-C PROGRAM, Connector_USB:USB_C_Receptacle_GCT_USB4110, symbol Connector:USB_C_Receptacle_USB2.0_16P
- added R17, R18: 5.1k, Resistor_SMD:R_0402_1005Metric, symbol Device:R
- added R19: 33k, Resistor_SMD:R_0402_1005Metric, symbol Device:R
- added R20: 82k, Resistor_SMD:R_0402_1005Metric, symbol Device:R
- added SW2: BOOT, Button_Switch_SMD:SW_SPST_PTS645Sx43SMTR92, symbol Switch:SW_Push
- added U2: USBLC6-2SC6, Package_TO_SOT_SMD:SOT-23-6, symbol Power_Protection:USBLC6-2SC6
- J1, J10, J2, J3: footprint Connector_PinHeader_2.54mm:PinHeader_1x02_P2.54mm_Vertical -> Connector_Molex:Molex_Micro-Fit_3.0_43650-0224_1x02-1MP_P3.00mm_Vertical; MPN (none) -> 436500224; Manufacturer (none) -> Molex
- J4, J5: footprint Connector_PinHeader_2.54mm:PinHeader_1x03_P2.54mm_Vertical -> Connector_Molex:Molex_Micro-Fit_3.0_43650-0324_1x03-1MP_P3.00mm_Vertical; MPN (none) -> 436500324; Manufacturer (none) -> Molex
- J6: footprint Connector_PinHeader_2.54mm:PinHeader_1x04_P2.54mm_Vertical -> Connector_Molex:Molex_Micro-Fit_3.0_43650-0424_1x04-1MP_P3.00mm_Vertical; MPN (none) -> 436500424; Manufacturer (none) -> Molex
- J8: footprint Connector_PinHeader_2.54mm:PinHeader_1x06_P2.54mm_Vertical -> Connector_Molex:Molex_Micro-Fit_3.0_43650-0624_1x06-1MP_P3.00mm_Vertical; MPN (none) -> 436500624; Manufacturer (none) -> Molex
- J9: footprint Connector_PinHeader_2.54mm:PinHeader_1x08_P2.54mm_Vertical -> Connector_Molex:Molex_Micro-Fit_3.0_43650-0824_1x08-1MP_P3.00mm_Vertical; MPN (none) -> 436500824; Manufacturer (none) -> Molex
Connections:
- net +3V3: now also U1.95 (VDD33_USB), C13.1, SW2.1
- net GND: now also C12.2, C13.2, J11.A1 (GND), J11.A12 (GND), J11.B1 (GND), J11.B12 (GND), J11.SH (SHIELD), R17.2, R18.2, R20.2, U2.2 (GND)
- net VDDA: no longer U1.95 (VDD33_USB)
- net USB_VBUS_SENSE: now reaches U1.101 (PA9)
- net USB_VBUS_SENSE: now also R19.2, R20.1
- net USB_DM: now reaches U1.103 (PA11)
- net USB_DM: now also J11.A7 (D-), J11.B7 (D-), U2.1 (I/O1), U2.6 (I/O1)
- net USB_DP: now reaches U1.104 (PA12)
- net USB_DP: now also J11.A6 (D+), J11.B6 (D+), U2.3 (I/O2), U2.4 (I/O2)
- net BOOT0: now reaches R4.2, U1.138 (BOOT0)
- net BOOT0: now also SW2.2
- new net USB_CC1: J11.A5 (CC1), R17.1
- new net USB_CC2: J11.B5 (CC2), R18.1
- new net USB_VBUS: C12.1, J11.A4 (VBUS), J11.A9 (VBUS), J11.B4 (VBUS), J11.B9 (VBUS), R19.1, U2.5 (VBUS)
- no-connect marks 4 -> 6
Other:
- note added: "USB FIRMWARE UPLOAD (SELF-POWERED) Use a USB data cable and normal board power. Hold BOOT, tap RESET, release BOOT; connect with STM32CubeProgrammer USB. BOOT_ADD1 must select system memory (0x1FF0); keep SWD for recovery. VBUS stays separate from board supply. PA9 is GPIO cable sensing. Use forced USB device mode; GPIO sensing, not native VBUS comparator. All added parts use SMT solder joints; s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"

Commit message: Update four KiCad designs and include portable project libraries
Parts:
- removed R10: 10k, Resistor_SMD:R_0402_1005Metric, symbol Device:R
- added C14: 10uF 50V X7R, Capacitor_SMD:C_1210_3225Metric, symbol Device:C
- added C15, C17: 100nF 50V X7R, Capacitor_SMD:C_0603_1608Metric, symbol Device:C
- added C16: 1uF 16V X7R, Capacitor_SMD:C_0603_1608Metric, symbol Device:C
- added J12: FAN 1 - P12 PRO, Connector:FanPinHeader_1x04_P2.54mm_Vertical, symbol Connector_Generic:Conn_01x04
- added J13: FAN 2 - P12 PRO, Connector:FanPinHeader_1x04_P2.54mm_Vertical, symbol Connector_Generic:Conn_01x04
- added J14: 12V FAN POWER, Connector_JST:JST_XH_B2B-XH-A_1x02_P2.50mm_Vertical, symbol Connector_Generic:Conn_01x02
- added J15: COOLER, Connector_JST:JST_XH_B2B-XH-A_1x02_P2.50mm_Vertical, symbol Connector_Generic:Conn_01x02
- added R21, R22: 10k, Resistor_SMD:R_0603_1608Metric, symbol Device:R
- added R23: 100k, Resistor_SMD:R_0603_1608Metric, symbol Device:R
- added R24: 100, Resistor_SMD:R_0603_1608Metric, symbol Device:R
- added U3: SN74LVC2G07DBVR, Package_TO_SOT_SMD:SOT-23-6, symbol 74xGxx:74LVC2G07
- added U4: TPS22919DCKR, Package_TO_SOT_SMD:SOT-363_SC-70-6, symbol BrainPower:TPS22919DCK
- C1, decoupl_C1, decoupl_C2, decoupl_C3: footprint Capacitor_SMD:C_0402_1005Metric -> BrainReviewed:C_0402_1005Metric_Reviewed_7; JLCPCB URL (none) -> https://jlcpcb.com/partdetail/MurataElectronics-GRM155R71H1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; LCSC (none) -> C77020; MPN (none) -> GRM155R71H104KE14D; Manufacturer (none) -> Murata; Rating (none) -> 100nF 50V X7R
- C10: footprint Capacitor_SMD:C_0402_1005Metric -> BrainReviewed:C_0402_1005Metric_Reviewed_4; JLCPCB URL (none) -> https://jlcpcb.com/partdetail/MurataElectronics-GRM155R61A1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; LCSC (none) -> C76999; MPN (none) -> GRM155R61A105KE15D; Manufacturer (none) -> Murata; Rating (none) -> 1uF 10V X5R
- C11: footprint Capacitor_SMD:C_0402_1005Metric -> BrainReviewed:C_0402_1005Metric_Reviewed_4; JLCPCB URL (none) -> https://jlcpcb.com/partdetail/MurataElectronics-GRM155R71H1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; LCSC (none) -> C77020; MPN (none) -> GRM155R71H104KE14D; Manufacturer (none) -> Murata; Rating (none) -> 100nF 50V X7R
- C12: footprint Capacitor_SMD:C_0402_1005Metric -> BrainReviewed:C_0402_1005Metric_Reviewed_3; JLCPCB URL (none) -> https://jlcpcb.com/partdetail/MurataElectronics-GRM155R71H1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; LCSC (none) -> C77020
- C13: footprint Capacitor_SMD:C_0402_1005Metric -> BrainReviewed:C_0402_1005Metric_Reviewed_3; JLCPCB URL (none) -> https://jlcpcb.com/partdetail/MurataElectronics-GRM155R61A1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; LCSC (none) -> C76999
- C2: footprint Capacitor_SMD:C_0402_1005Metric -> BrainReviewed:C_0402_1005Metric_Reviewed_2; JLCPCB URL (none) -> https://jlcpcb.com/partdetail/MurataElectronics-GRM155R71H1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; LCSC (none) -> C77020; MPN (none) -> GRM155R71H104KE14D; Manufacturer (none) -> Murata; Rating (none) -> 100nF 50V X7R
- C3: footprint Capacitor_SMD:C_0402_1005Metric -> BrainReviewed:C_0402_1005Metric_Reviewed_10; JLCPCB URL (none) -> https://jlcpcb.com/partdetail/MurataElectronics-GRM155R71H1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; LCSC (none) -> C77020; MPN (none) -> GRM155R71H104KE14D; Manufacturer (none) -> Murata; Rating (none) -> 100nF 50V X7R
- C4: footprint Capacitor_SMD:C_0402_1005Metric -> BrainReviewed:C_0402_1005Metric_Reviewed_8; JLCPCB URL (none) -> https://jlcpcb.com/partdetail/MurataElectronics-GRM1555C1H2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; LCSC (none) -> C76959; MPN (none) -> GRM1555C1H200JA01D; Manufacturer (none) -> Murata; Rating (none) -> 20pF 50V C0G
- C5: footprint Capacitor_SMD:C_0402_1005Metric -> BrainReviewed:C_0402_1005Metric_Reviewed_4; JLCPCB URL (none) -> https://jlcpcb.com/partdetail/MurataElectronics-GRM1555C1H2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; LCSC (none) -> C76959; MPN (none) -> GRM1555C1H200JA01D; Manufacturer (none) -> Murata; Rating (none) -> 20pF 50V C0G
- C6: footprint Capacitor_SMD:C_0402_1005Metric -> BrainReviewed:C_0402_1005Metric_Reviewed_9; JLCPCB URL (none) -> https://jlcpcb.com/partdetail/MurataElectronics-GRM155R71H1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; LCSC (none) -> C77020; MPN (none) -> GRM155R71H104KE14D; Manufacturer (none) -> Murata; Rating (none) -> 100nF 50V X7R
- C7: footprint Capacitor_SMD:C_0402_1005Metric -> BrainReviewed:C_0402_1005Metric_Reviewed_6; JLCPCB URL (none) -> https://jlcpcb.com/partdetail/MurataElectronics-GRM155R61A2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; LCSC (none) -> C77002; MPN (none) -> GRM155R61A225KE95D; Manufacturer (none) -> Murata; Rating (none) -> 2.2uF 10V X5R; Release Status (none) -> HOLD: verify effective capacitance and ESR at VCAP bias
- C8: footprint Capacitor_SMD:C_0402_1005Metric -> BrainReviewed:C_0402_1005Metric_Reviewed_12; JLCPCB URL (none) -> https://jlcpcb.com/partdetail/MurataElectronics-GRM1555C1H1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; LCSC (none) -> C76946; MPN (none) -> GRM1555C1H100JA01D; Manufacturer (none) -> Murata; Rating (none) -> 10pF 50V C0G
- C9: footprint Capacitor_SMD:C_0402_1005Metric -> BrainReviewed:C_0402_1005Metric_Reviewed_4; JLCPCB URL (none) -> https://jlcpcb.com/partdetail/MurataElectronics-GRM1555C1H1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; LCSC (none) -> C76946; MPN (none) -> GRM1555C1H100JA01D; Manufacturer (none) -> Murata; Rating (none) -> 10pF 50V C0G
- FB1: JLCPCB URL (none) -> https://jlcpcb.com/partdetail/MurataElectronics-BLM15AG601S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; LCSC (none) -> C76884; MPN (none) -> BLM15AG601SN1D; Manufacturer (none) -> Murata; Rating (none) -> 600 ohm at 100MHz; verify analog-rail DC drop
- J1, J10, J2: footprint Connector_Molex:Molex_Micro-Fit_3.0_43650-0224_1x02-1MP_P3.00mm_Vertical -> Connector_JST:JST_XH_B2B-XH-A_1x02_P2.50mm_Vertical; MPN 436500224 -> B2B-XH-A(LF)(SN); Manufacturer Molex -> JST (XH-compatible clone OK)
- J11: JLCPCB URL (none) -> https://jlcpcb.com/partdetail/5762033-USB4110_GFA/C5143397; LCSC (none) -> C5143397
- J3: value Conn_01x02 -> LEVEL SENSOR - ADAFRUIT 4965; footprint Connector_Molex:Molex_Micro-Fit_3.0_43650-0224_1x02-1MP_P3.00mm_Vertical -> Connector_JST:JST_XH_B3B-XH-A_1x03_P2.50mm_Vertical; symbol Connector_Generic:Conn_01x02 -> Connector_Generic:Conn_01x03; Cable Contact (none) -> SXH-001T-P0.6; MPN 436500224 -> B3B-XH-A(LF)(SN); Manufacturer Molex -> JST (XH-compatible clone OK); Mating Housing (none) -> XHP-3; Replacement Review (none) -> JST XH 2.50mm vertical THT, hand-soldered (Taiss XH kit, Am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; Selection Notes (none) -> JST XH 2.50mm vertical THT, hand-soldered (Taiss XH kit, Am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; Sourcing Status (none) -> JST XH 2.50mm vertical THT, hand-soldered (Taiss XH kit, Am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
- J4, J5: footprint Connector_Molex:Molex_Micro-Fit_3.0_43650-0324_1x03-1MP_P3.00mm_Vertical -> Connector_JST:JST_XH_B3B-XH-A_1x03_P2.50mm_Vertical; Cable Contact (none) -> SXH-001T-P0.6; MPN 436500324 -> B3B-XH-A(LF)(SN); Manufacturer Molex -> JST (XH-compatible clone OK); Mating Housing (none) -> XHP-3; Replacement Review (none) -> JST XH 2.50mm vertical THT, hand-soldered (Taiss XH kit, Am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; Selection Notes (none) -> JST XH 2.50mm vertical THT, hand-soldered (Taiss XH kit, Am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; Sourcing Status (none) -> JST XH 2.50mm vertical THT, hand-soldered (Taiss XH kit, Am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
- J6: footprint Connector_Molex:Molex_Micro-Fit_3.0_43650-0424_1x04-1MP_P3.00mm_Vertical -> Connector_JST:JST_XH_B4B-XH-A_1x04_P2.50mm_Vertical; MPN 436500424 -> B4B-XH-A(LF)(SN); Manufacturer Molex -> JST (XH-compatible clone OK)
- J7: JLCPCB URL (none) -> https://jlcpcb.com/partdetail/WurthElektronik-61301411121/C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; LCSC (none) -> C5907899; MPN (none) -> 61301411121; Manufacturer (none) -> Wurth Elektronik; Release Status (none) -> HOLD: confirm header drawing / exposed height with LCD/debu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
- J8: value Conn_01x06 -> LIGHT BOARD; footprint Connector_Molex:Molex_Micro-Fit_3.0_43650-0624_1x06-1MP_P3.00mm_Vertical -> Connector_JST:JST_XH_B5B-XH-A_1x05_P2.50mm_Vertical; symbol Connector_Generic:Conn_01x06 -> Connector_Generic:Conn_01x05; MPN 436500624 -> B5B-XH-A(LF)(SN); Manufacturer Molex -> JST (XH-compatible clone OK); Replacement Review (none) -> JST XH 2.50mm vertical THT, hand-soldered (Taiss XH kit, Am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; Selection Notes (none) -> JST XH 2.50mm vertical THT, hand-soldered (Taiss XH kit, Am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; Sourcing Status (none) -> JST XH 2.50mm vertical THT, hand-soldered (Taiss XH kit, Am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
- J9: value Conn_01x08 -> PUMP BOARD; footprint Connector_Molex:Molex_Micro-Fit_3.0_43650-0824_1x08-1MP_P3.00mm_Vertical -> Connector_JST:JST_XH_B6B-XH-A_1x06_P2.50mm_Vertical; symbol Connector_Generic:Conn_01x08 -> Connector_Generic:Conn_01x06; MPN 436500824 -> B6B-XH-A(LF)(SN); Manufacturer Molex -> JST (XH-compatible clone OK); Replacement Review (none) -> 8-circuit vertical through-hole Micro-Fit. Replace SMT foot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; Selection Notes (none) -> Vertical Micro-Fit replacement; PCB footprint updated where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; Sourcing Status (none) -> Catalog checked for 3 boards of each design; stock not rese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
- R1, R2, R3: footprint Resistor_SMD:R_0402_1005Metric -> BrainReviewed:R_0402_1005Metric_Reviewed_2; JLCPCB URL (none) -> https://jlcpcb.com/partdetail/YAGEO-RC0402FR071KL/C106235; LCSC (none) -> C106235; MPN (none) -> RC0402FR-071KL; Manufacturer (none) -> Yageo; Rating (none) -> 1%, 0402, 1/16W
- R11, R12, R13, R14, R15, R16, R4: footprint Resistor_SMD:R_0402_1005Metric -> BrainReviewed:R_0402_1005Metric_Reviewed_1; JLCPCB URL (none) -> https://jlcpcb.com/partdetail/YAGEO-RC0402FR0710KL/C60490; LCSC (none) -> C60490; MPN (none) -> RC0402FR-0710KL; Manufacturer (none) -> Yageo; Rating (none) -> 1%, 0402, 1/16W
- R17, R18: footprint Resistor_SMD:R_0402_1005Metric -> BrainReviewed:R_0402_1005Metric_Reviewed_5; JLCPCB URL (none) -> https://jlcpcb.com/partdetail/YAGEO-RC0402FR075K1L/C105872; LCSC (none) -> C105872
- R19: footprint Resistor_SMD:R_0402_1005Metric -> BrainReviewed:R_0402_1005Metric_Reviewed_6; JLCPCB URL (none) -> https://jlcpcb.com/partdetail/YAGEO-RC0402FR0733KL/C138003; LCSC (none) -> C138003
- R20: footprint Resistor_SMD:R_0402_1005Metric -> BrainReviewed:R_0402_1005Metric_Reviewed_4; JLCPCB URL (none) -> https://jlcpcb.com/partdetail/YAGEO-RC0402FR0782KL/C137932; LCSC (none) -> C137932
- R5: footprint Resistor_SMD:R_0402_1005Metric -> BrainReviewed:R_0402_1005Metric_Reviewed_1; JLCPCB URL (none) -> https://jlcpcb.com/partdetail/YAGEO-RC0402FR074K7L/C105871; LCSC (none) -> C105871; MPN (none) -> RC0402FR-074K7L; Manufacturer (none) -> Yageo; Rating (none) -> 1%, 0402, 1/16W
- R6: footprint Resistor_SMD:R_0402_1005Metric -> BrainReviewed:R_0402_1005Metric_Reviewed_6; JLCPCB URL (none) -> https://jlcpcb.com/partdetail/YAGEO-RC0402FR074K7L/C105871; LCSC (none) -> C105871; MPN (none) -> RC0402FR-074K7L; Manufacturer (none) -> Yageo; Rating (none) -> 1%, 0402, 1/16W
- R7, R8: value 1.9k -> 1.91k; footprint Resistor_SMD:R_0402_1005Metric -> BrainReviewed:R_0402_1005Metric_Reviewed_2; JLCPCB URL (none) -> https://jlcpcb.com/partdetail/YAGEO-RC0402FR071K91L/C477598; LCSC (none) -> C477598; MPN (none) -> RC0402FR-071K91L; Manufacturer (none) -> YAGEO; Rating (none) -> 1.91kohm, 1%, 0402, 62.5mW; Replacement Review (none) -> 1.91kohm 1% 0402 replaces 1.9kohm I2C pullups R7/R8. Nomina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; Sourcing Status (none) -> Catalog checked for 3 boards of each design; stock not rese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
- R9: footprint Resistor_SMD:R_0402_1005Metric -> BrainReviewed:R_0402_1005Metric_Reviewed_3; JLCPCB URL (none) -> https://jlcpcb.com/partdetail/YAGEO-RC0402FR0747RL/C137973; LCSC (none) -> C137973; MPN (none) -> RC0402FR-0747RL; Manufacturer (none) -> Yageo; Rating (none) -> 1%, 0402, 1/16W
- SW1: JLCPCB URL (none) -> https://jlcpcb.com/partdetail/CK-PTS645SM43SMTR92LFS/C221880; LCSC (none) -> C221880; MPN (none) -> PTS645SM43SMTR92 LFS; Manufacturer (none) -> C&K; Rating (none) -> SMT push switch
- SW2: JLCPCB URL (none) -> https://jlcpcb.com/partdetail/CK-PTS645SM43SMTR92LFS/C221880; LCSC (none) -> C221880
- SWDdebugHeader1: JLCPCB URL (none) -> https://jlcpcb.com/partdetail/WurthElektronik-61300411121/C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; LCSC (none) -> C5184785; MPN (none) -> 61300411121; Manufacturer (none) -> Wurth Elektronik; Release Status (none) -> HOLD: confirm header drawing / exposed height with LCD/debu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
- U1: JLCPCB URL (none) -> https://jlcpcb.com/partdetail/STMicroelectronics-STM32H753Z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; LCSC (none) -> C730207; MPN (none) -> STM32H753ZIT6; Manufacturer (none) -> STMicroelectronics; Rating (none) -> LQFP144, -40 to 85C
- U2: JLCPCB URL (none) -> https://jlcpcb.com/partdetail/STMicroelectronics-USBLC62SC6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; LCSC (none) -> C7519
- UARTdebugHeader1: JLCPCB URL (none) -> https://jlcpcb.com/partdetail/WurthElektronik-61300311121/C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; LCSC (none) -> C2915006; MPN (none) -> 61300311121; Manufacturer (none) -> Wurth Elektronik; Release Status (none) -> HOLD: confirm header drawing / exposed height with LCD/debu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
- VCAP_C1: footprint Capacitor_SMD:C_0402_1005Metric -> BrainReviewed:C_0402_1005Metric_Reviewed_1; JLCPCB URL (none) -> https://jlcpcb.com/partdetail/MurataElectronics-GRM155R61A2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; LCSC (none) -> C77002; MPN (none) -> GRM155R61A225KE95D; Manufacturer (none) -> Murata; Rating (none) -> 2.2uF 10V X5R; Release Status (none) -> HOLD: verify effective capacitance and ESR at VCAP bias
- Y1: footprint Crystal:Crystal_SMD_3225-4Pin_3.2x2.5mm -> BrainReviewed:Crystal_SMD_3225-4Pin_3.2x2.5mm_Reviewed_1; JLCPCB URL (none) -> https://jlcpcb.com/partdetail/ECS-ECS_80_12_33_JGNTR/C24426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; LCSC (none) -> C2442665; MPN (none) -> ECS-80-12-33-JGN-TR; Manufacturer (none) -> ECS; Rating (none) -> 8MHz, CL=12pF, ESR max 400 ohm; Release Status (none) -> HOLD: HSE gain margin / drive and sourcing; C4/C5 20pF impl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; Replacement Review (none) -> 8MHz, 12pF, 3225 four-pad crystal, 400-ohm ESR. Matches nom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; Sourcing Status (none) -> Catalog checked for 3 boards of each design; stock not rese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
- Y2: footprint Crystal:Crystal_SMD_3215-2Pin_3.2x1.5mm -> BrainReviewed:Crystal_SMD_3215-2Pin_3.2x1.5mm_Reviewed_1; JLCPCB URL (none) -> https://jlcpcb.com/partdetail/AbraconLLC-ABS07_32_768KHZ_7T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; LCSC (none) -> C276424; MPN (none) -> ABS07-32.768KHZ-7-T; Manufacturer (none) -> Abracon; Rating (none) -> 32.768kHz, CL=7pF; Release Status (none) -> HOLD: LSE drive/startup and sourcing; C8/C9 10pF imply 2pF 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
- decoupl_C10, decoupl_C8, decoupl_C9: footprint Capacitor_SMD:C_0402_1005Metric -> BrainReviewed:C_0402_1005Metric_Reviewed_1; JLCPCB URL (none) -> https://jlcpcb.com/partdetail/MurataElectronics-GRM155R71H1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; LCSC (none) -> C77020; MPN (none) -> GRM155R71H104KE14D; Manufacturer (none) -> Murata; Rating (none) -> 100nF 50V X7R
- decoupl_C11, decoupl_C12: footprint Capacitor_SMD:C_0402_1005Metric -> BrainReviewed:C_0402_1005Metric_Reviewed_13; JLCPCB URL (none) -> https://jlcpcb.com/partdetail/MurataElectronics-GRM155R71H1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; LCSC (none) -> C77020; MPN (none) -> GRM155R71H104KE14D; Manufacturer (none) -> Murata; Rating (none) -> 100nF 50V X7R
- decoupl_C13: footprint Capacitor_SMD:C_0402_1005Metric -> BrainReviewed:C_0402_1005Metric_Reviewed_5; JLCPCB URL (none) -> https://jlcpcb.com/partdetail/MurataElectronics-GRM155R71H1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; LCSC (none) -> C77020; MPN (none) -> GRM155R71H104KE14D; Manufacturer (none) -> Murata; Rating (none) -> 100nF 50V X7R
- decoupl_C4, decoupl_C5, decoupl_C7: footprint Capacitor_SMD:C_0402_1005Metric -> BrainReviewed:C_0402_1005Metric_Reviewed_6; JLCPCB URL (none) -> https://jlcpcb.com/partdetail/MurataElectronics-GRM155R71H1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; LCSC (none) -> C77020; MPN (none) -> GRM155R71H104KE14D; Manufacturer (none) -> Murata; Rating (none) -> 100nF 50V X7R
- decoupl_C6: footprint Capacitor_SMD:C_0402_1005Metric -> BrainReviewed:C_0402_1005Metric_Reviewed_11; JLCPCB URL (none) -> https://jlcpcb.com/partdetail/MurataElectronics-GRM155R71H1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; LCSC (none) -> C77020; MPN (none) -> GRM155R71H104KE14D; Manufacturer (none) -> Murata; Rating (none) -> 100nF 50V X7R
- rescaps_C1, rescaps_C2: footprint Capacitor_SMD:C_0402_1005Metric -> BrainReviewed:C_0402_1005Metric_Reviewed_7; JLCPCB URL (none) -> https://jlcpcb.com/partdetail/404009-GRM155R60J106ME15D/C41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; LCSC (none) -> C412251; MPN (none) -> GRM155R60J106ME15D; Manufacturer (none) -> Murata; Rating (none) -> 10uF 6.3V X5R; Release Status (none) -> HOLD: sourcing and effective 3.3V bulk capacitance verifica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
Connections:
- net +3V3: now also C15.1, C16.1, R21.1, R22.1, U3.5 (VCC), U4.1 (VIN)
- net COOLER: now also J15.1 (Pin_1); no longer J9.3 (Pin_3)
- net FAN_PWM: now also R21.2, U3.1; no longer J8.6 (Pin_6)
- net FLORA_BLOOM: now also J9.6 (Pin_6); no longer J9.8 (Pin_8)
- net FLORA_GROW: now also J9.5 (Pin_5); no longer J9.7 (Pin_7)
- net FLORA_MICRO: now also J9.4 (Pin_4); no longer J9.6 (Pin_6)
- net GND: now also C14.2, C15.2, C16.2, C17.2, J12.1 (Pin_1), J13.1 (Pin_1), J14.2 (Pin_2), J15.2 (Pin_2), R23.2, U3.2 (GND), U4.2 (GND)
- net LEVEL_PWR: now also R23.1, U4.3 (ON)
- net PH_DOWN: now also J9.3 (Pin_3); no longer J9.5 (Pin_5)
- net PH_UP: now also J9.2 (Pin_2); no longer J9.4 (Pin_4)
- net FAN2_PWM: now reaches U1.134 (PB4)
- net FAN2_PWM: now also R22.2, U3.3
- net HEATER: no longer names the net of U1.58 (PE7)
- net HEATER: no longer J9.2 (Pin_2)
- new net FAN1_CTL: J12.4 (Pin_4), U3.6
- new net FAN2_CTL: J13.4 (Pin_4), U3.4
- new net FAN_12V: C14.1, J12.2 (Pin_2), J13.2 (Pin_2), J14.1 (Pin_1)
- new net LEVEL_3V3: C17.1, J3.3 (Pin_3), R24.2, U4.6 (VOUT)
- new net LEVEL_DISCHG: R24.1, U4.5 (QOD)
- no-connect marks 6 -> 76
Other:
- note added: "ADAFRUIT 4965 WATER DETECTION J3: 1 = S (LEVEL_IN), 2 = - (GND), 3 = + (switched 3V3). PG2 / LEVEL_PWR enables U4: high = sensor powered. U4 QOD discharges sensor supply when disabled; R23 defaults OFF. Sensor output is wet/dry indication, not calibrated depth. Existing signal stays on PC3_C through R3/C3. Firmware owner: verify ADC3 channel / PC3_C analog switch; PA3 is unwired."
- note added: "DS3231_RTC"
- note added: "J15 COOLER -> power board J6 (1 COOL_EN, 2 GND) J9 -> pump board J1, pin-for-pin"
- note added: "PA3 is unused on this PCB. Level input is PC3_C / ADC3_INP1. Reviewed: readWaterLevel uses hadc3; MX_ADC3_Init selects channel 1; MSP opens SYSCFG_SWITCH_PC3. Legacy PA3 ADC2 initialization may be removed by firmware owner."
- note added: "PWMConnector"
- note added: "TWO INDEPENDENT FANS: PE14 / TIM1_CH4 and PB4 / TIM3_CH1. U3 preserves PWM polarity; outputs use the fan internal pull-ups. R21/R22 pull MCU-side controls to 3V3; default released input = full speed. J14: protected 12V from power-board J7. Never connect to J10 (3V3). J12/J13 pin 3 tachometer unused. Firmware maintained by teammate."
- note added: "enclosureTempProbe"
- note added: "powerIn"
- note added: "pumpConnector"
- note added: "screenConnector"
- note added: "waterTempProbe"
