File: pump_PCB/pump_PCB.kicad_pcb (KiCad board)
At the start: 2 copper layers, 138 x 85 mm, 52 parts, among them J1 CONTROL INPUT, J2 POWER INPUT, J3 FLORA_GROW, J4 FLORA_BLOOM, J5 FLORA_MICRO, J6 PH_UP, J7 PH_DOWN, M1 CSD18540Q5B, M2 CSD18540Q5B, M3 CSD18540Q5B, M4 CSD18540Q5B, M5 CSD18540Q5B, U1 TC4420CPA, U2 TC4420CPA, U3 TC4420CPA, U4 TC4420CPA, U5 TC4420CPA

Commit message: Update four KiCad designs and include portable project libraries
Parts:
- C1, C10, C2, C3, C4, C5, C6, C7, C8, C9: footprint Capacitor_THT:C_Disc_D3.8mm_W2.6mm_P2.50mm -> Capacitor_SMD:C_0603_1608Metric
- J1: footprint Connector_Molex:Molex_Micro-Fit_3.0_43650-0624_1x06-1MP_P3.00mm_Vertical -> Connector_JST:JST_XH_B6B-XH-A_1x06_P2.50mm_Vertical
- J2: footprint Connector_Molex:Molex_Micro-Fit_3.0_43650-0324_1x03-1MP_P3.00mm_Vertical -> Connector_JST:JST_XH_B3B-XH-A_1x03_P2.50mm_Vertical
- J3, J4, J5, J6, J7: footprint Connector_Molex:Molex_Micro-Fit_3.0_43650-0224_1x02-1MP_P3.00mm_Vertical -> Connector_JST:JST_XH_B2B-XH-A_1x02_P2.50mm_Vertical
- moved J1 6.99 mm to (34.2, 95.0)
- moved J2 4.01 mm to (24.0, 45.5)
- moved J3 3.38 mm to (66.8, 26.0)
- moved J4 3.38 mm to (92.8, 26.0)
- moved J5 3.38 mm to (40.8, 26.0)
- moved J6 3.38 mm to (118.8, 26.0)
- moved J7 3.38 mm to (144.8, 26.0)
- moved C1 1.25 mm to (29.2, 60.5)
- moved C10 1.25 mm to (139.2, 60.5)
- moved C2 1.25 mm to (55.2, 60.5)
- moved C3 1.25 mm to (81.2, 60.5)
- moved C4 1.25 mm to (107.2, 60.5)
- moved C5 1.25 mm to (133.2, 60.5)
- moved C6 1.25 mm to (35.2, 60.5)
- moved C7 1.25 mm to (61.2, 60.5)
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Routing:
- net /+12V: track 495.9 -> 501.3 mm
- net /GND: track 27.4 -> 32.2 mm, vias 38 -> 48
Other:
- board text added: "HYDROPONIC PUMPS"
- board text removed: "12V | COMMON GND"
- board text removed: "PUMP DRIVER REV A"
